File: RC_Demo_Elec/motor_driver_stage.kicad_sch (KiCad schematic)
At the start: 6 parts, among them Q1 IRF9540N, Q2 2N7000

Commit message: [chore] - pin ThetOS to v1.1.0 + commit Cargo.lock + schematic added note
Changed lines of the file:
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@@
+		)
+	)
+	(text_box "SW_EN driven by PWM"
+		(exclude_from_sim no)
+		(at 133.35 74.7917 0)
+		(size 24.13 3.9483)
+		(margins 0.9525 0.9525 0.9525 0.9525)
+		(stroke
+			(width 0)
+			(type solid)
+		)
+		(fill
+			(type none)
+		)
+		(effects
+			(font
+				(size 1.27 1.27)
+			)
+			(justify left top)
 		)
 	)
@@
 		)
 	)
-	(sheet_instances
-		(path "/"
-			(page "1")
-		)
-	)
-	(embedded_fonts no)
 )

Commit message: [refactor] - forwards made 100% duty + 1K pullup in schematic motor
Parts:
- R2, R4: value 10K -> 1K
